File: shield/shield.brd (EAGLE design)
At the start: 102.5 x 66 mm, 18 parts, among them IC1 LM75, Q1 IPP114N03L, U1 TLC5925IDWR

Commit message: Update for manufacturing
Connections:
- net +3V3: no longer SV2.4, SV2.5, SV3.3, SV3.4, SV3.5, SV3.6
- net GND: no longer SV1.11, SV1.22, SV1.5, SV2.14, SV2.15, SV2.26, SV2.30, SV2.43, SV2.48, SV2.52, SV2.57, SV2.79, SV3.19, SV3.55, SV3.66, SV3.73
Routing:
- net +3V3: track 265.1 -> 197.5 mm
- net GND: track 169.1 -> 218.4 mm
- net P48: track 25.5 -> 27.4 mm
- net P77: track 88.7 -> 88.0 mm
- removed copper zone on layer 1, net GND

Commit message: update
Parts:
- moved D1 3.81 mm to (77.5, 45.7)
- moved Q1 3.81 mm to (74.9, 54.6)
- moved LED1 2.54 mm to (83.8, 62.2)
- moved R3 2.54 mm to (73.7, 63.5)
- moved R5 2.54 mm to (73.7, 59.7)
- moved DIS2 1.91 mm to (22.9, 33.7)
Connections:
- net P74: now also U1.21
- net P77: no longer LED1.A, Q1.G, R3.2
- net P80: no longer U1.21
- net P83: now also LED1.A, Q1.G, R3.2
Routing:
- net P77: track 88.0 -> 0.00 mm
- net P83: track 0.00 -> 80.1 mm
- net P80: track 69.2 -> 0.00 mm, vias 1 -> 0
- net P74: track 0.00 -> 65.6 mm
- net P48: track 27.4 -> 35.6 mm
- net P41: track 53.4 -> 61.3 mm
- net N$11: track 84.1 -> 90.0 mm
- net +3V3: track 197.5 -> 201.9 mm
- net N$17: track 29.1 -> 25.7 mm
- net N$9: track 36.3 -> 38.2 mm
- net N$8: track 5.49 -> 7.39 mm
- net N$7: track 8.55 -> 10.5 mm
- net N$6: track 12.4 -> 14.3 mm
- net N$5: track 32.5 -> 34.4 mm
- net N$2: track 64.2 -> 66.1 mm
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