File: shield/shield.sch (EAGLE design)
At the start: 18 parts, among them IC1 LM75, Q1 IPP114N03L, U1 TLC5925IDWR

Commit message: Update for manufacturing
Connections:
- net +3V3: no longer SV2.4, SV2.5, SV3.3, SV3.4, SV3.5, SV3.6
- net GND: no longer SV1.11, SV1.22, SV1.5, SV2.14, SV2.15, SV2.26, SV2.30, SV2.43, SV2.48, SV2.52, SV2.57, SV2.79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

Commit message: update
Connections:
- net P74: now also U1.~OE
- net P77: no longer LED1.A, Q1.G, R3.2
- net P80: no longer U1.~OE
- net P83: now also LED1.A, Q1.G, R3.2
